File: hardware/heater-controller/heater-controller.kicad_sch (KiCad schematic)
At the start: 36 parts, among them J1 JST-XH 5P, J4 USB_C_Receptacle_USB2.0_14P, SW1 SW_Push, SW2 SW_Push, U1 TPS54202DDC, U2 ESP32-S3-MINI-1-N8R2, U4 TCAN332, U5 AP2112K-3.3

Commit message: Add protected analog/mixed and digital IO connectors
J2 (analog/mixed) breaks out ADC1 pins IO1-4, IO7-10 with IO8/IO9 marked
as I2C SDA/SCL; J3 (digital) breaks out IO11-18 with SPI on IO11-14 and
UART1 on IO17/18. Both are 10-pin JST-XH with fused 3V3 and GND, and
every line has a 1k series resistor and an SRV05-4 clamp. Analog lines
get a 10nF filter cap; I2C pull-ups are fitted as DNP. Sheet moves to A3.

Also adds the initial PCB file created from the earlier schematic.

Co-Authored-By: Claude Opus 5.5 <noreply@anthropic.com>
Parts:
- added C14, C15, C16, C17, C18, C19: 10nF, Capacitor_SMD:C_0603_1608Metric, symbol Device:C
- added F2, F3: 200mA PTC, Fuse:Fuse_1206_3216Metric, symbol Device:Polyfuse
- added J2: Analog / Mixed IO, Connector_JST:JST_XH_B10B-XH-A_1x10_P2.50mm_Vertical, symbol Connector_Generic:Conn_01x10
- added J3: Digital IO, Connector_JST:JST_XH_B10B-XH-A_1x10_P2.50mm_Vertical, symbol Connector_Generic:Conn_01x10
- added R14, R15, R16, R17, R18, R19, R21, R23, R24, R25, R26, R27, R28, R29, R30, R31: 1k, Resistor_SMD:R_0603_1608Metric, symbol Device:R
- added R20, R22: 4.7k, Resistor_SMD:R_0603_1608Metric, symbol Device:R
- added U6, U7, U8, U9: SRV05-4, Package_TO_SOT_SMD:SOT-23-6, symbol Power_Protection:SRV05-4
Connections:
- net +3.3V: now also F2.1, F3.1, R20.1, R22.1, U6.5 (VP), U7.5 (VP), U8.5 (VP), U9.5 (VP)
- net GND: now also C14.2, C15.2, C16.2, C17.2, C18.2, C19.2, J2.10 (Pin_10), J3.10 (Pin_10), U6.2 (VN), U7.2 (VN), U8.2 (VN), U9.2 (VN)
- net IO7: now reaches U2.11 (IO7)
- net IO7: now also C18.1, R18.1
- net IO8_SDA: now reaches U2.12 (IO8)
- net IO8_SDA: now also R19.1, R20.2
- net IO9_SCL: now reaches U2.13 (IO9)
- net IO9_SCL: now also R21.1, R22.2
- net IO10: now reaches U2.14 (IO10)
- net IO10: now also C19.1, R23.1
- net IO11_MOSI: now reaches U2.15 (IO11)
- net IO11_MOSI: now also R24.1
- net IO12_SCK: now reaches U2.16 (IO12)
- net IO12_SCK: now also R25.1
- net IO13_MISO: now reaches U2.17 (IO13)
- net IO13_MISO: now also R26.1
- net IO14_CS: now reaches U2.18 (IO14)
- net IO14_CS: now also R27.1
- net IO15: now reaches U2.19 (IO15)
- net IO15: now also R28.1
- net IO16: now reaches U2.20 (IO16)
- net IO16: now also R29.1
- net IO17_TX1: now reaches U2.21 (IO17)
- net IO17_TX1: now also R30.1
- net IO18_RX1: now reaches U2.22 (IO18)
- net IO18_RX1: now also R31.1
- net IO1: now reaches U2.5 (IO1)
- net IO1: now also C14.1, R14.1
- net IO2: now reaches U2.6 (IO2)
- net IO2: now also C15.1, R15.1
- net IO3: now reaches U2.7 (IO3)
- net IO3: now also C16.1, R16.1
- net IO4: now reaches U2.8 (IO4)
- net IO4: now also C17.1, R17.1
- new net J2_3V3: F2.2, J2.1 (Pin_1)
- new net J2_IO1: J2.2 (Pin_2), R14.2, U6.1 (IO1)
- new net J2_IO10: J2.9 (Pin_9), R23.2, U7.6 (IO4)
- new net J2_IO2: J2.3 (Pin_3), R15.2, U6.3 (IO2)
- new net J2_IO3: J2.4 (Pin_4), R16.2, U6.4 (IO3)
- new net J2_IO4: J2.5 (Pin_5), R17.2, U6.6 (IO4)
- new net J2_IO7: J2.6 (Pin_6), R18.2, U7.1 (IO1)
- new net J2_IO8_SDA: J2.7 (Pin_7), R19.2, U7.3 (IO2)
- new net J2_IO9_SCL: J2.8 (Pin_8), R21.2, U7.4 (IO3)
- new net J3_3V3: F3.2, J3.1 (Pin_1)
- new net J3_IO11_MOSI: J3.2 (Pin_2), R24.2, U8.1 (IO1)
- new net J3_IO12_SCK: J3.3 (Pin_3), R25.2, U8.3 (IO2)
- new net J3_IO13_MISO: J3.4 (Pin_4), R26.2, U8.4 (IO3)
- new net J3_IO14_CS: J3.5 (Pin_5), R27.2, U8.6 (IO4)
- new net J3_IO15: J3.6 (Pin_6), R28.2, U9.1 (IO1)
- new net J3_IO16: J3.7 (Pin_7), R29.2, U9.3 (IO2)
- new net J3_IO17_TX1: J3.8 (Pin_8), R30.2, U9.4 (IO3)
- new net J3_IO18_RX1: J3.9 (Pin_9), R31.2, U9.6 (IO4)
- no-connect marks 35 -> 19
Other:
- note added: "Analog / Mixed IO (J2)"
- note added: "Digital IO (J3)"
- note added: "J2: 1 3V3 (fused) 2 IO1 3 IO2 4 IO3 5 IO4 6 IO7 7 IO8 I2C SDA 8 IO9 I2C SCL 9 IO10 10 GND. All ADC1 (usable with Wi-Fi). 1k series + SRV05-4 clamp on every line. 10nF filter on analog lines; 4.7k I2C pull-ups DNP. IO3 is a strapping pin (JTAG select, only if the eFuse is set)."
- note added: "J3: 1 3V3 (fused) 2 IO11 SPI MOSI 3 IO12 SPI SCK 4 IO13 SPI MISO 5 IO14 SPI CS 6 IO15 7 IO16 8 IO17 UART1 TX 9 IO18 UART1 RX 10 GND. 1k series + SRV05-4 clamp on every line (keep SPI to ~4 MHz). ADC2 pins: no analog while Wi-Fi is on."
